File: cao_00/cao/button.kicad_sch (KiCad schematic)
At the start: 2 parts, among them SW2 SW_Push

Commit message: added footprint
Parts:
- R1: renamed from R2; footprint (none) -> footprint:R
- SW1: renamed from SW2; footprint (none) -> footprint:SW_PUSH
Changed lines of the file:
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@@
   (symbol (lib_id "power:GND") (at 51.435 45.085 0)
     (in_bom yes) (on_board yes) (fields_autoplaced)
-    (property "Reference" "#PWR0121" (id 0) (at 51.435 51.435 0)
+    (property "Reference" "#PWR0119" (id 0) (at 51.435 51.435 0)
       (effects (font (size 1.27 1.27)) hide)
     )
@@
   (symbol (lib_id "New_Library:R") (at 53.34 31.75 270)
     (in_bom yes) (on_board yes)
-    (property "Reference" "R2" (id 0) (at 53.34 30.4799 90)
+    (property "Reference" "R1" (id 0) (at 53.34 30.4799 90)
       (effects (font (size 1.27 1.27)) (justify left))
     )
@@
       (effects (font (size 1.27 1.27)) (justify left))
     )
-    (property "Footprint" "" (id 2) (at 53.34 31.75 0)
+    (property "Footprint" "footprint:R" (id 2) (at 53.34 31.75 0)
       (effects (font (size 1.27 1.27)) hide)
     )
@@
   (symbol (lib_id "power:+5V") (at 51.435 28.575 0)
     (in_bom yes) (on_board yes) (fields_autoplaced)
-    (property "Reference" "#PWR0122" (id 0) (at 51.435 32.385 0)
+    (property "Reference" "#PWR0120" (id 0) (at 51.435 32.385 0)
       (effects (font (size 1.27 1.27)) hide)
     )
@@
   (symbol (lib_id "New_Library:SW_Push") (at 51.435 40.005 270)
     (in_bom yes) (on_board yes) (fields_autoplaced)
-    (property "Reference" "SW2" (id 0) (at 55.88 38.7349 90)
+    (property "Reference" "SW1" (id 0) (at 55.88 38.7349 90)
       (effects (font (size 1.27 1.27)) (justify left))
     )
@@
       (effects (font (size 1.27 1.27)) (justify left))
     )
-    (property "Footprint" "" (id 2) (at 56.515 40.005 0)
+    (property "Footprint" "footprint:SW_PUSH" (id 2) (at 56.515 40.005 0)
       (effects (font (size 1.27 1.27)) hide)
     )
