File: cao_00/cao/cao.kicad_sch (KiCad schematic)
At the start: 8 parts, among them J2 AVR-ISP-6, U1 ATmega328P-AU, Y1 16MHz

Commit message: added footprint
Parts:
- C1, C2, C4, C5: footprint (none) -> footprint:C_0603
- H1: footprint (none) -> footprint:MountingHole_2.1mm
- J2: footprint (none) -> footprint:AVR-ISP-6
- U1: footprint (none) -> footprint:ATMEGA328P_AU
- Y1: footprint (none) -> footprint:CRISTAL_16MH
Changed lines of the file:
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@@
       (effects (font (size 1.27 1.27)) (justify right))
     )
-    (property "Footprint" "" (id 2) (at 158.115 57.15 90)
+    (property "Footprint" "footprint:AVR-ISP-6" (id 2) (at 158.115 57.15 90)
       (effects (font (size 1.27 1.27)) hide)
     )
@@
       (effects (font (size 1 1)))
     )
-    (property "Footprint" "" (id 2) (at 82.55 71.12 0)
+    (property "Footprint" "footprint:CRISTAL_16MH" (id 2) (at 82.55 71.12 0)
       (effects (font (size 1.27 1.27)) hide)
     )
@@
       (effects (font (size 1.27 1.27)) (justify left))
     )
-    (property "Footprint" "" (id 2) (at 62.23 45.72 0)
+    (property "Footprint" "footprint:ATMEGA328P_AU" (id 2) (at 62.23 45.72 0)
       (effects (font (size 1.27 1.27)) hide)
     )
@@
       (effects (font (size 1.27 1.27)) (justify left))
     )
-    (property "Footprint" "" (id 2) (at 154.94 121.92 0)
+    (property "Footprint" "footprint:MountingHole_2.1mm" (id 2) (at 154.94 121.92 0)
       (effects (font (size 1.27 1.27)) hide)
     )
@@
       (effects (font (size 1.27 1.27)) (justify right))
     )
-    (property "Footprint" "" (id 2) (at 78.74 73.66 0)
+    (property "Footprint" "footprint:C_0603" (id 2) (at 78.74 73.66 0)
       (effects (font (size 1.27 1.27)) hide)
     )
@@
       (effects (font (size 1.27 1.27)) (justify left))
     )
-    (property "Footprint" "" (id 2) (at 86.36 73.66 0)
+    (property "Footprint" "footprint:C_0603" (id 2) (at 86.36 73.66 0)
       (effects (font (size 1.27 1.27)) hide)
     )
@@
       (effects (font (size 1.27 1.27)) (justify right))
     )
-    (property "Footprint" "" (id 2) (at 67.31 33.02 0)
+    (property "Footprint" "footprint:C_0603" (id 2) (at 67.31 33.02 0)
       (effects (font (size 1.27 1.27)) hide)
     )
@@
       (effects (font (size 1.27 1.27)) (justify left))
     )
-    (property "Footprint" "" (id 2) (at 72.39 33.02 0)
+    (property "Footprint" "footprint:C_0603" (id 2) (at 72.39 33.02 0)
       (effects (font (size 1.27 1.27)) hide)
     )
@@
     )
     (path "/68cff6c3-e6b5-403e-830c-8d37d3a66595"
-      (reference "C1") (unit 1) (value "22pF") (footprint "")
+      (reference "C1") (unit 1) (value "22pF") (footprint "footprint:C_0603")
     )
     (path "/775cc646-5f97-4229-a318-626f6c8e7a95"
-      (reference "C2") (unit 1) (value "22pF") (footprint "")
+      (reference "C2") (unit 1) (value "22pF") (footprint "footprint:C_0603")
     )
     (path "/31e60d74-5801-46c1-a0c2-7a6f7a34faf5/abf3ea9c-902a-4506-81ce-aa0bc4d7c315"
-      (reference "C3") (unit 1) (value "100nF") (footprint "")
+      (reference "C3") (unit 1) (value "100nF") (footprint "footprint:C_0603")
     )
     (path "/b8725906-0027-4fe7-960d-1fdba3862dec"
-      (reference "C4") (unit 1) (value "100nF") (footprint "")
+      (reference "C4") (unit 1) (value "100nF") (footprint "footprint:C_0603")
     )
     (path "/77cf35d5-4a0e-4ffc-a559-cbffedf79299"
-      (reference "C5") (unit 1) (value "10uF") (footprint "")
+      (reference "C5") (unit 1) (value "10uF") (footprint "footprint:C_0603")
     )
     (path "/26f37cc8-f6bd-4572-9f9a-8d95eb1bf505/b16ffba1-740b-49c8-af97-87b9c12d2290"
-      (reference "D1") (unit 1) (value "LED") (footprint "")
+      (reference "D1") (unit 1) (value "LED") (footprint "footprint:LED_0603")
     )
     (path "/0e41cc12-1035-443a-a68f-63b7d17be7de/b16ffba1-740b-49c8-af97-87b9c12d2290"
-      (reference "D2") (unit 1) (value "LED") (footprint "")
+      (reference "D2") (unit 1) (value "LED") (footprint "footprint:LED_0603")
     )
     (path "/842ef6f7-1429-4475-acdc-3be0591e3637/b16ffba1-740b-49c8-af97-87b9c12d2290"
-      (reference "D3") (unit 1) (value "LED") (footprint "")
+      (reference "D3") (unit 1) (value "LED") (footprint "footprint:LED_0603")
     )
     (path "/42bb59ad-7076-45a5-89e3-ad287e0808fc/b16ffba1-740b-49c8-af97-87b9c12d2290"
-      (reference "D4") (unit 1) (value "LED") (footprint "")
+      (reference "D4") (unit 1) (value "LED") (footprint "footprint:LED_0603")
     )
     (path "/21ce9945-d928-416c-b855-ec0ddffa5b8a"
-      (reference "H1") (unit 1) (value "MountingHole") (footprint "")
+      (reference "H1") (unit 1) (value "MountingHole") (footprint "footprint:MountingHole_2.1mm")
     )
     (path "/31e60d74-5801-46c1-a0c2-7a6f7a34faf5/85c487df-11b6-4056-94ab-bb21457133a8"
-      (reference "J1") (unit 1) (value "Conn_01x06") (footprint "")
+      (reference "J1") (unit 1) (value "Conn_01x06") (footprint "footprint:Conn_01x06")
     )
     (path "/09758c59-e622-4004-ba9d-7b17699af83f"
-      (reference "J2") (unit 1) (value "AVR-ISP-6") (footprint "")
+      (reference "J2") (unit 1) (value "AVR-ISP-6") (footprint "footprint:AVR-ISP-6")
     )
     (path "/b4eab0d6-c29a-4eb7-9bad-3341dcf434e2/3f4e9dc1-0c75-47a0-838f-76420603ef83"
-      (reference "R1") (unit 1) (value "10K") (footprint "")
+      (reference "R1") (unit 1) (value "10K") (footprint "footprint:R")
     )
     (path "/90b213b1-2044-47f1-89e2-0460c750aa06/3f4e9dc1-0c75-47a0-838f-76420603ef83"
-      (reference "R2") (unit 1) (value "10K") (footprint "")
+      (reference "R2") (unit 1) (value "10K") (footprint "footprint:R")
     )
     (path "/26f37cc8-f6bd-4572-9f9a-8d95eb1bf505/7e380278-8c67-4e2e-b992-175205a39d6e"
-      (reference "R3") (unit 1) (value "330R") (footprint "")
+      (reference "R3") (unit 1) (value "330R") (footprint "footprint:R")
     )
     (path "/0e41cc12-1035-443a-a68f-63b7d17be7de/7e380278-8c67-4e2e-b992-175205a39d6e"
-      (reference "R4") (unit 1) (value "330R") (footprint "")
+      (reference "R4") (unit 1) (value "330R") (footprint "footprint:R")
     )
     (path "/842ef6f7-1429-4475-acdc-3be0591e3637/7e380278-8c67-4e2e-b992-175205a39d6e"
-      (reference "R5") (unit 1) (value "330R") (footprint "")
+      (reference "R5") (unit 1) (value "330R") (footprint "footprint:R")
     )
     (path "/42bb59ad-7076-45a5-89e3-ad287e0808fc/7e380278-8c67-4e2e-b992-175205a39d6e"
-      (reference "R6") (unit 1) (value "330R") (footprint "")
+      (reference "R6") (unit 1) (value "330R") (footprint "footprint:R")
     )
     (path "/b4eab0d6-c29a-4eb7-9bad-3341dcf434e2/f8a2c7df-9f05-4caf-a85b-8675b8b89d37"
-      (reference "SW1") (unit 1) (value "SW_Push") (footprint "")
+      (reference "SW1") (unit 1) (value "SW_Push") (footprint "footprint:SW_PUSH")
     )
     (path "/90b213b1-2044-47f1-89e2-0460c750aa06/f8a2c7df-9f05-4caf-a85b-8675b8b89d37"
-      (reference "SW2") (unit 1) (value "SW_Push") (footprint "")
+      (reference "SW2") (unit 1) (value "SW_Push") (footprint "footprint:SW_PUSH")
     )
     (path "/1c16c01b-0823-44f7-bd11-f50b59eca726"
-      (reference "U1") (unit 1) (value "ATmega328P-AU") (footprint "")
+      (reference "U1") (unit 1) (value "ATmega328P-AU") (footprint "footprint:ATMEGA328P_AU")
     )
     (path "/0b6c0cf5-d5a3-45a6-9f17-6486abf9c013"
-      (reference "Y1") (unit 1) (value "16MHz") (footprint "")
-    )
-  )
+      (reference "Y1") (unit 1) (value "16MHz") (footprint "footprint:CRISTAL_16MH")
+    )
+  )
