File: cao_00/cao/led.kicad_sch (KiCad schematic)
At the start: 2 parts

Commit message: added footprint
Parts:
- D4: footprint (none) -> footprint:LED_0603
- R6: footprint (none) -> footprint:R
Changed lines of the file:
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@@
     (property "Reference" "R6" (id 0) (at 55.88 37.465 0))
     (property "Value" "330R" (id 1) (at 55.88 39.37 0))
-    (property "Footprint" "" (id 2) (at 55.88 40.005 0)
+    (property "Footprint" "footprint:R" (id 2) (at 55.88 40.005 0)
       (effects (font (size 1.27 1.27)) hide)
     )
@@
       (effects (font (size 1.27 1.27)) hide)
     )
-    (property "Footprint" "" (id 2) (at 46.355 41.91 0)
+    (property "Footprint" "footprint:LED_0603" (id 2) (at 46.355 41.91 0)
       (effects (font (size 1.27 1.27)) hide)
     )
