File: cao_00/cao/usb_flasher.kicad_sch (KiCad schematic)
At the start: 2 parts, among them J1 Conn_01x06

Commit message: added footprint
Parts:
- C3: footprint (none) -> footprint:C_0603
- J1: footprint (none) -> footprint:Conn_01x06
Changed lines of the file:
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@@
     (property "Reference" "J1" (id 0) (at 30.48 23.495 0))
     (property "Value" "Conn_01x06" (id 1) (at 27.305 32.385 90))
-    (property "Footprint" "" (id 2) (at 31.115 31.115 0)
+    (property "Footprint" "footprint:Conn_01x06" (id 2) (at 31.115 31.115 0)
       (effects (font (size 1.27 1.27)) hide)
     )
@@
       (effects (font (size 1 1)))
     )
-    (property "Footprint" "" (id 2) (at 38.735 36.195 0)
+    (property "Footprint" "footprint:C_0603" (id 2) (at 38.735 36.195 0)
       (effects (font (size 1.27 1.27)) hide)
     )
