File: cao_00/cao/cao.kicad_pcb (KiCad board)
At the start: 2 copper layers, 22 parts, among them J1 Conn_01x06, J2 AVR-ISP-6, SW1 SW_Push, SW2 SW_Push, U1 ATmega328P-AU, Y1 16MHz

Commit message: last backup
Connections:
- R1 pad 2: (no net) -> GND
- R2 pad 1: (no net) -> GND
- R2 pad 2: (no net) -> /BUT_0
Routing:
- net GND: track 62.2 -> 84.9 mm, vias 0 -> 2
- net /BUT_0: track 0.00 -> 5.64 mm
- net +5V: track 42.5 -> 43.9 mm
- added copper zone on B.Cu, net GND
- added copper zone on F.Cu, net GND
